File: smiw-pcb/dom_panel/PWR_LINE.kicad_sch (KiCad schematic)
At the start: 6 parts, among them J2 Barrel_Jack_Switch, U4 PT4115, U5 REG1117A

Commit message: wsszystko
Parts:
- added U10: mp1584_module, symbol mp1584_module:mp1584_module
- added U6: LM3410XMF, LM3410XMF:SOT95P280X145-5N, symbol LM3410XMF:LM3410XMF
Connections:
- net +12V: now also U10.1 (IN2+), U10.2 (IN+)
- net +3V3: now also U10.5 (OUT+), U10.6 (OUT2+)
- net GND: now also U10.3 (IN-), U10.4 (IN2-), U10.7 (OUT-), U10.8 (OUT2-), U6.2 (GND); no longer U4.2 (GND)
Other:
- moved on the sheet: D1, L1, R1, U4
